File: hardware/CADENCE_SWANS/Payload/Payload Controller/Prototype_Payload_Controller/Payload_Controller_EM.kicad_pcb (KiCad board)
At the start: 4 copper layers, 98 x 100 mm, 126 parts, among them J1 Conn_01x06_Pin, J11 Conn_01x04, J12 Conn_01x02, J13 USB_C_Receptacle_USB2.0_16P, J14 Conn_01x02, J15 Conn_02x02_Top_Bottom, J2 Conn_01x06_Pin, J3 Conn_01x06_Pin, J4 Conn_01x06_Pin, J5 Conn_Coaxial, J6 Conn_Coaxial, J7 Conn_Coaxial, J8 Conn_Coaxial, J9 Conn_01x02, SW1 KMR2, SW2 KMR2, U1 SN65C1168ERGYR, U25 LSM6DSO, U27 LIS2MDL, U29 TMP112xxDRL, U3 LT8612, U31 INA219AxDCN, U5 LT8612, U6 LT8612, U8 ATSAMV71Q21B-A, Y1 ABM3B-12.000MHZ-B2-T, Y2 ABS07-32.768KHZ-T

Commit message: Schematic/PCB Corrections and Ready To Export
Parts:
- added G***: LOGO, LOGO, B.Cu at (171.2, 119.6)
- added G***: LOGO, LOGO, B.Cu at (182.1, 119.2)
- C44, C45, C51, C52: footprint Capacitor_SMD:C_0805_2012Metric -> Capacitor_SMD:C_1206_3216Metric
- J4: moved to F.Cu
- moved J4 4.03 mm to (109.0, 73.3), turned to 180 degrees
- moved R121 2.58 mm to (150.9, 123.7), turned to 180 degrees
- moved C51 1.85 mm to (125.4, 106.7)
- moved C52 1.07 mm to (122.5, 106.7)
- moved C45 1.04 mm to (124.7, 119.4)
- moved C44 0.43 mm to (121.9, 119.5)
Connections:
- C19 pad 1: +3V3 -> +3.3V
- C20 pad 2: +3V3 -> +3.3V
- C24 pad 1: +3V3 -> +3.3V
- C39 pad 1: VBAT -> VBAT_SYS
- C46 pad 1: VBAT -> VBAT_SYS
- C7 pad 1: VBAT -> VBAT_SYS
- L1 pad 2: +3V3 -> +3.3V
- R121 pad 2: +3.3V -> VBAT_SYS
- R6 pad 2: +3V3 -> +3.3V
- TP10 pad 1: VBAT -> VBAT_SYS
- TP4 pad 1: VBAT -> VBAT_SYS
- TP7 pad 1: VBAT -> VBAT_SYS
- TP9 pad 1: +3V3 -> +3.3V
- U3 pad 4: VBAT -> VBAT_SYS
- U3 pad 5: VBAT -> VBAT_SYS
- U3 pad 6: VBAT -> VBAT_SYS
- U3 pad 7: VBAT -> VBAT_SYS
- U31 pad 2: +3.3V -> VBAT_SYS
- U31 pad 4: VBAT -> +3.3V
- U5 pad 4: VBAT -> VBAT_SYS
- U5 pad 5: VBAT -> VBAT_SYS
- U5 pad 6: VBAT -> VBAT_SYS
- U5 pad 7: VBAT -> VBAT_SYS
- U6 pad 22: +3V3 -> +3.3V
- U6 pad 4: VBAT -> VBAT_SYS
- U6 pad 5: VBAT -> VBAT_SYS
- U6 pad 6: VBAT -> VBAT_SYS
- U6 pad 7: VBAT -> VBAT_SYS
Routing:
- net +12V: track 227.4 -> 360.2 mm, vias 17 -> 20
- net VBAT_SYS: track 0.00 -> 117.3 mm, vias 0 -> 2
- net +3.3V: track 61.1 -> 133.6 mm, vias 3 -> 5
- net VBAT: track 180.7 -> 154.5 mm
- net /Instrument/CTRL_EN_4: track 47.3 -> 42.4 mm
- net +3V3: track 93.3 -> 89.8 mm, vias 28 -> 25
- net /Instrument/CTRL_R1_4: track 45.8 -> 47.6 mm
- net GND: track 127.5 -> 126.1 mm
- net +5V: track 138.3 -> 139.4 mm
- net /Instrument/CTRL_EN_3: track 65.9 -> 67.0 mm
- net /Instrument/CTRL_R2_4: track 53.5 -> 54.4 mm
Other:
- board text added: "Angelo Duenas Pragun Bethapudi"
- board text added: "Payload Controller"
- board text removed: "if only reuse blocks existed in KiCAD..."
