File: hardware/CADENCE_SWANS/Payload/Payload Controller/Prototype_Payload_Controller/power_management.kicad_sch (KiCad schematic)
At the start: 57 parts, among them U3 LT8612, U31 INA219AxDCN, U5 LT8612, U6 LT8612

Commit message: Schematic/PCB Corrections and Ready To Export
Parts:
- C44, C45, C51, C52: footprint Capacitor_SMD:C_0805_2012Metric -> Capacitor_SMD:C_1206_3216Metric
Connections:
- net +3V3 is gone; now on net +3.3V: C19.1, C20.2, C24.1, L1.2, R6.2, TP9.1, U6.22 (BIAS)
- net +3.3V: now also U31.4 (VS); no longer R121.2, U31.2 (IN-)
- net VBAT: no longer C39.1, C46.1, C7.1, TP10.1, TP4.1, TP7.1, U3.4 (EN/UV), U3.5 (VIN), U3.6 (VIN), U3.7 (VIN), U31.4 (VS), U5.4 (EN/UV), U5.5 (VIN), U5.6 (VIN), U5.7 (VIN), U6.4 (EN/UV), U6.5 (VIN), U6.6 (VIN), U6.7 (VIN)
- new net VBAT_SYS: C39.1, C46.1, C7.1, R121.2, TP10.1, TP4.1, TP7.1, U3.4 (EN/UV), U3.5 (VIN), U3.6 (VIN), U3.7 (VIN), U31.2 (IN-), U5.4 (EN/UV), U5.5 (VIN), U5.6 (VIN), U5.7 (VIN), U6.4 (EN/UV), U6.5 (VIN), U6.6 (VIN), U6.7 (VIN)
